File: mic_pcb.kicad_pcb (KiCad board)
At the start: 2 copper layers, 36.5 x 63 mm, 24 parts, among them J1 MIC_IN, J2 GAIN, J3 AUDIO_OUT, J4 5v USB, Q1 2N4416, U1 THAT1512, U2 NMA0515SC

Commit message: Add files via upload
updated design
Routing:
- net Net-(C6-Pad2): track 41.7 -> 33.5 mm
- net Net-(C2-Pad1): track 42.1 -> 35.4 mm
- net Net-(C1-Pad1): track 30.7 -> 24.9 mm
- net Net-(J2-Pad2): track 21.4 -> 16.0 mm
- net Net-(C6-Pad1): track 34.7 -> 39.6 mm
- net Net-(C2-Pad2): track 53.4 -> 50.1 mm, vias 2 -> 0
- net Net-(C1-Pad2): track 59.1 -> 56.5 mm
- net Net-(C5-Pad2): track 65.3 -> 67.4 mm, vias 1 -> 0
- net Net-(J2-Pad1): track 17.3 -> 16.4 mm
